File: soylent.sch (KiCad schematic (older format))
At the start: 17 parts, among them J1 DB9_Female, J2 Conn_01x04, J3 Conn_01x04, J4 Conn_02x03_Counter_Clockwise, Q1 BC847BPN, U1 ATtiny202-SS, U2 MIC5504-3.3YM5

Commit message: Route regulator
Parts:
- JP1, JP2: footprint (none) -> Jumpers:SMT-JUMPER_2_NO_SILK
Changed lines of the file:
@@
 F 0 "JP1" H 6500 4913 50  0000 C CNN
 F 1 "SolderJumper_2_Open" H 6500 4914 50  0001 C CNN
-F 2 "" H 6500 4800 50  0001 C CNN
+F 2 "Jumpers:SMT-JUMPER_2_NO_SILK" H 6500 4800 50  0001 C CNN
 F 3 "~" H 6500 4800 50  0001 C CNN
 	1    6500 4800
@@
 F 0 "JP2" H 7850 5113 50  0000 C CNN
 F 1 "SolderJumper_2_Bridged" H 7850 5114 50  0001 C CNN
-F 2 "" H 7850 5000 50  0001 C CNN
+F 2 "Jumpers:SMT-JUMPER_2_NO_SILK" H 7850 5000 50  0001 C CNN
 F 3 "~" H 7850 5000 50  0001 C CNN
 	1    7850 5000
